File: PicoChainATtiny85/PicoChainATtiny85.kicad_sch (KiCad schematic)
At the start: 11 parts, among them J1 RJ45, J2 RJ45, J3 Servo, U1 LM78M05_TO252, U2 PCA9615DP, U3 ATtiny85-20P, U4 LM78M05_TO252

Commit message: Added licences and PDF schematics
Other:
- title: (none) -> PicoChainATtiny85 Reference Device Implementation
Changed lines of the file:
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@@
 	(generator_version "8.0")
 	(paper "A4")
+	(title_block
+		(title "PicoChainATtiny85 Reference Device Implementation")
+		(date "2024-08-22")
+		(rev "v1.1")
+		(comment 2 "http://www.tapr.org/OHL")
+		(comment 3 "Licence: The TAPR Open Hardware License")
+		(comment 4 "Author: Jason Alexander")
+	)
 	(junction
 		(at 132.08 57.15)
