File: PicoChainTerminator/PicoChainTerminator.kicad_pcb (KiCad board)
At the start: 2 copper layers, 17 x 32 mm, 10 parts, among them J1 RJ45, U1 LM78M05

Commit message: Updated to 1.2
Parts:
- moved C1 1.24 mm to (96.2, 86.1)
- moved C2 1.24 mm to (91.6, 86.1)
- moved U1 1.24 mm to (93.9, 94.9)
- moved R2 1.24 mm to (101.9, 95.1)
- moved R3 1.24 mm to (101.9, 93.2)
- moved J1 1.24 mm to (101.9, 79.5)
- moved R1 1.24 mm to (99.3, 94.0)
- moved R5 1.24 mm to (101.8, 86.3)
- moved R6 1.24 mm to (101.8, 88.2)
- moved R4 1.22 mm to (99.2, 87.2)
Connections:
- R1 pad 1: Net-(J1-Pad4) -> Net-(J1-Pad6)
- R2 pad 1: Net-(J1-Pad4) -> Net-(J1-Pad6)
- R4 pad 2: Net-(J1-Pad6) -> Net-(J1-Pad4)
- R6 pad 1: Net-(J1-Pad6) -> Net-(J1-Pad4)
Routing:
- net +5V: track 41.3 -> 32.5 mm, vias 0 -> 2
- net Net-(J1-Pad6): track 9.38 -> 17.0 mm, vias 0 -> 1
- net Net-(J1-Pad4): track 15.3 -> 8.75 mm, vias 1 -> 0
- net GND: vias 0 -> 4
- added copper zone on In1.Cu, net GND
- added copper zone on In2.Cu, net GND
Other:
- copper layers 2 -> 4
- board text added: "PicoDaisy (v1.2)"
- board text removed: "PicoDaisy (v1.1)"

Commit message: Finial changes before ordering first boards.
Parts:
- U1: value LM78M05 -> LM78M05_TO252
Changed lines of the file:
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@@
 			(psa4output no)
 			(plot_black_and_white yes)
-			(plotinvisibletext no)
 			(sketchpadsonfab no)
 			(plotpadnumbers no)
@@
 			)
 		)
-		(property "Datasheet" ""
+		(property "Datasheet" "~"
 			(at 0 0 0)
 			(unlocked yes)
@@
 			)
 		)
-		(property "Datasheet" ""
+		(property "Datasheet" "~"
 			(at 0 0 90)
 			(unlocked yes)
@@
 			)
 		)
-		(property "Datasheet" ""
+		(property "Datasheet" "~"
 			(at 0 0 90)
 			(unlocked yes)
@@
 			)
 		)
-		(property "Datasheet" ""
+		(property "Datasheet" "~"
 			(at 0 0 270)
 			(unlocked yes)
@@
 			)
 		)
-		(property "Value" "LM78M05"
+		(property "Value" "LM78M05_TO252"
 			(at -0.056 4.093 270)
 			(layer "F.SilkS")
@@
 			)
 		)
-		(property "Datasheet" ""
+		(property "Datasheet" "~"
 			(at 0 0 0)
 			(unlocked yes)
@@
 			)
 		)
-		(property "Datasheet" ""
+		(property "Datasheet" "~"
 			(at 0 0 0)
 			(unlocked yes)
@@
 			)
 		)
-		(property "Datasheet" ""
+		(property "Datasheet" "~"
 			(at 0 0 90)
 			(unlocked yes)
@@
 			)
 		)
-		(property "Datasheet" ""
+		(property "Datasheet" "~"
 			(at 0 0 180)
 			(unlocked yes)
@@
 			)
 		)
-		(property "Datasheet" ""
+		(property "Datasheet" "~"
 			(at 0 0 0)
 			(unlocked yes)
