File: PicoChainZero/PicoChainZero.kicad_pcb (KiCad board)
At the start: 4 copper layers, 68 x 50 mm, 37 parts, among them J1 RJ45, J2 RJ45, J3 Raspberry Pi, J4 USB_C_Receptacle_USB2.0_14P, J5 +12V In, J6 +24V In, U1 LM78M05, U2 FT232RL, U3 SRV05, U4 PCA9615DP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

Commit message: Added decoupling capacitors to dI2C drivers (doh)
Parts:
- added C8: 10uF, Capacitor_Tantalum_SMD:CP_EIA-3216-18_Kemet-A, F.Cu at (104.4, 73.6)
- added C9: 10uF, Capacitor_Tantalum_SMD:CP_EIA-3216-18_Kemet-A, F.Cu at (126.7, 67.6)
Routing:
- net +5V: track 170.6 -> 178.9 mm
- net +12V: track 71.3 -> 73.8 mm

Commit message: Adjustments to PicoChainZero
Parts:
- added J7: Conn_01x02_Pin, Connector_PinHeader_2.54mm:PinHeader_1x02_P2.54mm_Vertical, F.Cu at (148.3, 85.5)
- added J8: Conn_01x02_Pin, Connector_PinHeader_2.54mm:PinHeader_1x02_P2.54mm_Vertical, F.Cu at (102.2, 90.2)
Connections:
- J3 pad 14: unconnected-(J3-Pin_14-Pad14) -> GND
- J3 pad 20: unconnected-(J3-Pin_20-Pad20) -> GND
- J3 pad 25: unconnected-(J3-Pin_25-Pad25) -> GND
- J3 pad 30: unconnected-(J3-Pin_30-Pad30) -> GND
- J3 pad 34: unconnected-(J3-Pin_34-Pad34) -> GND
- J3 pad 6: unconnected-(J3-Pin_6-Pad6) -> GND
- J3 pad 9: unconnected-(J3-Pin_9-Pad9) -> GND
Routing:
- net +12V: track 73.8 -> 97.0 mm
- net Net-(J6-Pin_2): track 23.9 -> 36.0 mm
- net Net-(J5-Pin_2): track 46.7 -> 56.9 mm
- net Net-(C12-Pad2): track 5.21 -> 8.91 mm
- net Net-(C6-Pad2): track 5.22 -> 8.90 mm
- net +24V: track 70.2 -> 73.2 mm

Commit message: Finial changes before ordering first boards.
Parts:
- removed the C8 at (104.4, 73.6)
- added C13: 10uF, Capacitor_SMD:C_0805_2012Metric, F.Cu at (104.5, 72.8)
- renumbered C9 to C8
Connections:
- J4 pad A1: GND -> Net-(J4-SHIELD)
- J4 pad A12: GND -> Net-(J4-SHIELD)
- J4 pad B1: GND -> Net-(J4-SHIELD)
- J4 pad B12: GND -> Net-(J4-SHIELD)
Routing:
- net Net-(J4-SHIELD): track 19.5 -> 25.2 mm
